Commit message: Added Body and Leg assembly macros

File: robot/millihex.xacro (robot description, xacro)
@@ -45,6 +45,6 @@
     </joint>
   </xacro:macro>
-  <!-- Leg Definition -->
-  <xacro:macro name="shoulder" params="number">
+  <!-- Leg Link Definition -->
+  <xacro:macro name="millihex_link" params="number">
     <link name="shoulder${number}">
       <inertial>
@@ -56,14 +56,20 @@
         <origin xyz="0 0 0.00025" rpy="0 0 0"/>
         <geometry>
-          <box size="0.14 0.04 0.0005" />
+          <box size="0.03 0.02 0.0005" />
         </geometry>
       </collision>
       <visual>
-        <origin rpy="0.0 0 0" xyz="0 0 0"/>
+        <origin rpy="0 0 0" xyz="0 0 0"/>
         <geometry>
-          <box size="0.14 0.04 0.0005" />
+          <box size="0.03 0.02 0.0005" />
         </geometry>
       </visual>
     </link>
+  </xacro:macro>
+  <!-- Assemble Body -->
+  <xacro:macro name="millihex_body" params="">
+  </xacro:macro>
+  <!-- Assemble Leg -->
+  <xacro:macro name="millihex_leg" params="">
   </xacro:macro>
   <!-- Add Control -->

Commit message: Added leg joint transmission macro

File: robot/millihex.xacro (robot description, xacro)
@@ -46,6 +46,6 @@
   </xacro:macro>
   <!-- Leg Link Definition -->
-  <xacro:macro name="millihex_link" params="number">
-    <link name="shoulder${number}">
+  <xacro:macro name="millihex_link" params="leg_number joint_number">
+    <link name="leg${leg_number}_joint${joint_number}">
       <inertial>
         <origin xyz="0 0 0.00025" rpy="0 0 0" />
@@ -67,4 +67,17 @@
     </link>
   </xacro:macro>
+  <!-- Leg Joint Transmission -->
+  <xacro:macro name="leg_transmission" params="leg_number joint_number">
+    <transmission name="leg${leg_number}_joint${joint_number}_tran">
+      <type>transmission_interface/SimpleTransmission</type>
+      <joint name="leg${leg_number}_joint${joint_number}">
+        <hardwareInterface>EffortJointInterface</hardwareInterface>
+      </joint>
+      <actuator name="leg${leg_number}_joint${joint_number}_motor">
+        <hardwareInterface>EffortJointInterface</hardwareInterface>
+        <mechanicalReduction>1</mechanicalReduction>
+      </actuator>
+    </transmission>
+  </xacro:macro>
   <!-- Assemble Body -->
   <xacro:macro name="millihex_body" params="">

Commit message: Outlining xacro and added robot link mass and dimension properties

File: robot/millihex.xacro (robot description, xacro)
@@ -2,9 +2,15 @@
 <robot xmlns:xacro="http://www.ros.org/wiki/xacro" name="millihex">
   <!-- Properties -->
-	<xacro:property name="foot_kp" value="1000.0"/>
-	<xacro:property name="foot_kd" value="1000.0"/>
-	<xacro:property name="foot_mu1" value="10.0"/>
-  <xacro:property name="foot_mu2" value="10.0"/>
-  <!-- Useful Math MACROS-->
+  <xacro:property name="torso_mass" value="0.01" />
+  <xacro:property name="torso_x" value="0.14" />
+  <xacro:property name="torso_y" value="0.04" />
+  <xacro:property name="leg_link_mass" value="0.0008" />
+  <xacro:property name="leg_link_x" value="0.03" />
+  <xacro:property name="leg_link_y" value="0.02" />
+  <xacro:property name="pcb_thickness_z" value="0.0005" />
+	<xacro:property name="foot_kp" value="1000.0" />
+	<xacro:property name="foot_kd" value="1000.0" />
+	<xacro:property name="foot_mu1" value="10.0" />
+  <xacro:property name="foot_mu2" value="10.0" />
   <!-- Calculate Moment of Inertia of Box -->
   <xacro:macro name="box_inertia" params="mass x y z">
@@ -19,7 +25,7 @@
     <link name="torso">
       <inertial>
-        <origin xyz="0 0 0.00025" rpy="0 0 0" />
-        <mass value="0.01" />
-        <xacro:box_inertia mass="0.01" x="0.14" y="0.04" z="0.0005" />
+        <origin xyz="0 0 ${pcb_thickness_z / 2}" rpy="0 0 0" />
+        <mass value="${torso_mass}" />
+        <xacro:box_inertia mass="${torso_mass}" x="0.14" y="0.04" z="0.0005" />
       </inertial>
       <collision>
@@ -36,8 +42,5 @@
       </visual>
     </link>
-    <gazebo reference="head_link">
-        <mu1>10.0</mu1>
-        <mu2>10.0</mu2>
-    </gazebo>
+    <!-- TODO: insert torso frictions -->
     <joint name="base_joint" type="fixed">
         <parent link="base_link"/>
@@ -46,15 +49,15 @@
   </xacro:macro>
   <!-- Leg Link Definition -->
-  <xacro:macro name="millihex_link" params="leg_number joint_number">
-    <link name="leg${leg_number}_joint${joint_number}">
+  <xacro:macro name="millihex_leg_link" params="leg_number link_number link_mass x_length y_length z_length">
+    <link name="leg${leg_number}_link${link_number}">
       <inertial>
-        <origin xyz="0 0 0.00025" rpy="0 0 0" />
+        <origin xyz="0 0 ${z_length / 2}" rpy="0 0 0" />
         <mass value="0.01" />
-        <xacro:box_inertia mass="0.0008" x="0.03" y="0.02" z="0.0005" />
+        <xacro:box_inertia mass="0.0008" x="${x_length}" y="${y_length}" z="${z_length}" />
       </inertial>
       <collision>
         <origin xyz="0 0 0.00025" rpy="0 0 0"/>
         <geometry>
-          <box size="0.03 0.02 0.0005" />
+          <box size="0.02 0.03 0.0005" />
         </geometry>
       </collision>
@@ -62,8 +65,9 @@
         <origin rpy="0 0 0" xyz="0 0 0"/>
         <geometry>
-          <box size="0.03 0.02 0.0005" />
+          <box size="0.02 0.03 0.0005" />
         </geometry>
       </visual>
     </link>
+    <!-- TODO: insert link frictions -->
   </xacro:macro>
   <!-- Leg Joint Transmission -->
@@ -80,17 +84,31 @@
     </transmission>
   </xacro:macro>
+  <!-- Assemble Leg -->
+  <xacro:macro name="millihex_leg" params="leg_number">
+    <xacro:millihex_leg_link leg_number="" joint_number="" />
+    <joint name="leg${leg_number}_joint" type="fixed">
+      <parent link="lowerleg_M${number}_link"/>
+      <child link="footM${number}_link"/>
+      <origin xyz="0 0 0.06" rpy="0 0 0"/>
+    </joint>
+    <joint name="leg1_joint1" type="revolute">
+      <parent link="torso" />
+      <child link="leg1_link1" />
+      <origin xyz="0.08333333 -0.05 0" rpy="0 0 0" />
+      <limit lower="-1.5708" upper="1.5708" effort="1" velocity="1"/>
+      <axis xyz="1 0 0" />
+    </joint>
+  </xacro:macro>
   <!-- Assemble Body -->
-  <xacro:macro name="millihex_body" params="">
+  <xacro:macro name="millihex_body" params="leg_number joint_number">
+    <xacro:millihex_torso />
   </xacro:macro>
-  <!-- Assemble Leg -->
-  <xacro:macro name="millihex_leg" params="">
-  </xacro:macro>
-  <!-- Add Control -->
+  <!-- Add Gazebo Control Library -->
   <xacro:macro name="millihex_control" params="namespace">
-      <gazebo>
-          <plugin name="gazebo_ros_control" filename="libgazebo_ros_control.so">
-              <robotNamespace>/${namespace}</robotNamespace>
-          </plugin>
-      </gazebo>
+    <gazebo>
+      <plugin name="gazebo_ros_control" filename="libgazebo_ros_control.so">
+        <robotNamespace>/${namespace}</robotNamespace>
+      </plugin>
+    </gazebo>
   </xacro:macro>
   <!-- Build Robot by Filling in Macro Parameters -->

Commit message: Replaced hard-coded link geometries with generalized variables

File: robot/millihex.xacro (robot description, xacro)
@@ -27,16 +27,16 @@
         <origin xyz="0 0 ${pcb_thickness_z / 2}" rpy="0 0 0" />
         <mass value="${torso_mass}" />
-        <xacro:box_inertia mass="${torso_mass}" x="0.14" y="0.04" z="0.0005" />
+        <xacro:box_inertia mass="${torso_mass}" x="${torso_x}" y="${torso_y}" z="${pcb_thickness_z}" />
       </inertial>
       <collision>
-        <origin xyz="0 0 0.00025" rpy="0 0 0"/>
+        <origin xyz="0 0 ${pcb_thickness_z / 2}" rpy="0 0 0"/>
         <geometry>
-          <box size="0.14 0.04 0.0005" />
+          <box size="${torso_x} ${torso_y} ${pcb_thickness_z}" />
         </geometry>
       </collision>
       <visual>
-        <origin rpy="0.0 0 0" xyz="0 0 0"/>
+        <origin rpy="0 0 0" xyz="0 0 0"/>
         <geometry>
-          <box size="0.14 0.04 0.0005" />
+          <box size="${torso_x} ${torso_y} ${pcb_thickness_z}" />
         </geometry>
       </visual>
@@ -49,15 +49,15 @@
   </xacro:macro>
   <!-- Leg Link Definition -->
-  <xacro:macro name="millihex_leg_link" params="leg_number link_number link_mass x_length y_length z_length">
+  <xacro:macro name="millihex_leg_link" params="leg_number link_number x_length y_length">
     <link name="leg${leg_number}_link${link_number}">
       <inertial>
-        <origin xyz="0 0 ${z_length / 2}" rpy="0 0 0" />
-        <mass value="0.01" />
-        <xacro:box_inertia mass="0.0008" x="${x_length}" y="${y_length}" z="${z_length}" />
+        <origin xyz="0 0 ${pcb_thickness_z / 2}" rpy="0 0 0" />
+        <mass value="${leg_link_mass}" />
+        <xacro:box_inertia mass="0.0008" x="${x_length}" y="${y_length}" z="${pcb_thickness_z}" />
       </inertial>
       <collision>
-        <origin xyz="0 0 0.00025" rpy="0 0 0"/>
+        <origin xyz="0 0 ${pcb_thickness_z / 2}" rpy="0 0 0"/>
         <geometry>
-          <box size="0.02 0.03 0.0005" />
+          <box size="${x_length} ${y_length} ${pcb_thickness_z}" />
         </geometry>
       </collision>
@@ -65,5 +65,5 @@
         <origin rpy="0 0 0" xyz="0 0 0"/>
         <geometry>
-          <box size="0.02 0.03 0.0005" />
+          <box size="${x_length} ${y_length} ${pcb_thickness_z}" />
         </geometry>
       </visual>

Commit message: Updated joint definitions and created test assembly for robot body with 2 leg links and 1 moving leg joint

File: robot/millihex.xacro (robot description, xacro)
@@ -6,6 +6,6 @@
   <xacro:property name="torso_y" value="0.04" />
   <xacro:property name="leg_link_mass" value="0.0008" />
-  <xacro:property name="leg_link_x" value="0.03" />
-  <xacro:property name="leg_link_y" value="0.02" />
+  <xacro:property name="leg_link_x" value="0.02" />
+  <xacro:property name="leg_link_y" value="0.03" />
   <xacro:property name="pcb_thickness_z" value="0.0005" />
 	<xacro:property name="foot_kp" value="1000.0" />
@@ -54,5 +54,5 @@
         <origin xyz="0 0 ${pcb_thickness_z / 2}" rpy="0 0 0" />
         <mass value="${leg_link_mass}" />
-        <xacro:box_inertia mass="0.0008" x="${x_length}" y="${y_length}" z="${pcb_thickness_z}" />
+        <xacro:box_inertia mass="${leg_link_mass}" x="${x_length}" y="${y_length}" z="${pcb_thickness_z}" />
       </inertial>
       <collision>
@@ -86,21 +86,30 @@
   <!-- Assemble Leg -->
   <xacro:macro name="millihex_leg" params="leg_number">
-    <xacro:millihex_leg_link leg_number="" joint_number="" />
-    <joint name="leg${leg_number}_joint" type="fixed">
-      <parent link="lowerleg_M${number}_link"/>
-      <child link="footM${number}_link"/>
-      <origin xyz="0 0 0.06" rpy="0 0 0"/>
-    </joint>
-    <joint name="leg1_joint1" type="revolute">
-      <parent link="torso" />
-      <child link="leg1_link1" />
-      <origin xyz="0.08333333 -0.05 0" rpy="0 0 0" />
+    <!-- link 1 (shoulder link), horizontally oriented -->
+    <xacro:millihex_leg_link leg_number="${leg_number}" link_number="1"
+                             x_length="${leg_link_x}" y_length="${leg_link_y}" />
+    <!-- link 2, vertically oriented -->
+    <xacro:millihex_leg_link leg_number="${leg_number}" link_number="2"
+                             x_length="${leg_link_y}" y_length="${leg_link_x}" />
+    <joint name="leg${leg_number}_joint2" type="revolute">
+      <parent link="leg${leg_number}_link1" />
+      <child link="leg${leg_number}_link2" />
+      <origin xyz="-${leg_link_y} 0 0" rpy="0 0 0" />
       <limit lower="-1.5708" upper="1.5708" effort="1" velocity="1"/>
       <axis xyz="1 0 0" />
     </joint>
+    <xacro:leg_transmission leg_number="${leg_number}" joint_number="2" />
+    <!-- TODO: link 3, horizontally oriented -->
+    <!-- TODO: link 4, horizontally oriented -->
   </xacro:macro>
   <!-- Assemble Body -->
-  <xacro:macro name="millihex_body" params="leg_number joint_number">
+  <xacro:macro name="millihex_body" params="">
     <xacro:millihex_torso />
+    <xacro:millihex_leg leg_number="1" />
+    <joint name="leg1_joint1" type="fixed">
+      <parent link="torso" />
+      <child link="leg1_link1" />
+      <origin xyz="${torso_x / 2} ${torso_y / 2} 0" rpy="0 0 0" />
+    </joint>
   </xacro:macro>
   <!-- Add Gazebo Control Library -->
@@ -114,4 +123,5 @@
   <!-- Build Robot by Filling in Macro Parameters -->
   <xacro:millihex_torso />
+  <xacro:millihex_body />
   <xacro:millihex_control namespace="millihex" />
 </robot>

Commit message: Modified joint location orientations

File: robot/millihex.xacro (robot description, xacro)
@@ -95,5 +95,5 @@
       <parent link="leg${leg_number}_link1" />
       <child link="leg${leg_number}_link2" />
-      <origin xyz="-${leg_link_y} 0 0" rpy="0 0 0" />
+      <origin xyz="0 -${leg_link_x / 2 + leg_link_y / 2} 0" rpy="0 0 0" />
       <limit lower="-1.5708" upper="1.5708" effort="1" velocity="1"/>
       <axis xyz="1 0 0" />
@@ -110,5 +110,5 @@
       <parent link="torso" />
       <child link="leg1_link1" />
-      <origin xyz="${torso_x / 2} ${torso_y / 2} 0" rpy="0 0 0" />
+      <origin xyz="${torso_x / 2} -${torso_y / 2} 0" rpy="0 0 0" />
     </joint>
   </xacro:macro>

Commit message: Changed link colors and updated origin for link visual property

File: robot/millihex.xacro (robot description, xacro)
@@ -20,5 +20,5 @@
   </xacro:macro>
   <!-- Base and Torso Definition -->
-  <xacro:macro name="millihex_torso" params="">
+  <xacro:macro name="millihex_torso" params="color">
     <link name="base_link">
     </link>
@@ -36,5 +36,5 @@
       </collision>
       <visual>
-        <origin rpy="0 0 0" xyz="0 0 0"/>
+        <origin xyz="0 0 0" rpy="0 0 0" />
         <geometry>
           <box size="${torso_x} ${torso_y} ${pcb_thickness_z}" />
@@ -42,5 +42,11 @@
       </visual>
     </link>
-    <!-- TODO: insert torso frictions -->
+    <gazebo reference="torso">
+      <kp>${foot_kp}</kp>
+      <kd>${foot_kd}</kd>
+      <mu1>${foot_mu1}</mu1>
+      <mu2>${foot_mu2}</mu2>
+      <material>Gazebo/${color}</material>
+    </gazebo>
     <joint name="base_joint" type="fixed">
         <parent link="base_link"/>
@@ -49,5 +55,5 @@
   </xacro:macro>
   <!-- Leg Link Definition -->
-  <xacro:macro name="millihex_leg_link" params="leg_number link_number x_length y_length">
+  <xacro:macro name="millihex_leg_link" params="leg_number link_number x_length y_length color">
     <link name="leg${leg_number}_link${link_number}">
       <inertial>
@@ -63,5 +69,5 @@
       </collision>
       <visual>
-        <origin rpy="0 0 0" xyz="0 0 0"/>
+        <origin xyz="-${x_length / 2} -${y_length / 2} 0" rpy="0 0 0" />
         <geometry>
           <box size="${x_length} ${y_length} ${pcb_thickness_z}" />
@@ -69,5 +75,11 @@
       </visual>
     </link>
-    <!-- TODO: insert link frictions -->
+    <gazebo reference="leg${leg_number}_link${link_number}">
+      <kp>${foot_kp}</kp>
+      <kd>${foot_kd}</kd>
+      <mu1>${foot_mu1}</mu1>
+      <mu2>${foot_mu2}</mu2>
+      <material>Gazebo/${color}</material>
+    </gazebo>
   </xacro:macro>
   <!-- Leg Joint Transmission -->
@@ -88,14 +100,16 @@
     <!-- link 1 (shoulder link), horizontally oriented -->
     <xacro:millihex_leg_link leg_number="${leg_number}" link_number="1"
-                             x_length="${leg_link_x}" y_length="${leg_link_y}" />
+                             x_length="${leg_link_x}" y_length="${leg_link_y}"
+                             color="Black" />
     <!-- link 2, vertically oriented -->
     <xacro:millihex_leg_link leg_number="${leg_number}" link_number="2"
-                             x_length="${leg_link_y}" y_length="${leg_link_x}" />
+                             x_length="${leg_link_y}" y_length="${leg_link_x}"
+                             color="Orange" />
     <joint name="leg${leg_number}_joint2" type="revolute">
       <parent link="leg${leg_number}_link1" />
       <child link="leg${leg_number}_link2" />
-      <origin xyz="0 -${leg_link_x / 2 + leg_link_y / 2} 0" rpy="0 0 0" />
+      <origin xyz="0 -${leg_link_y} 0" rpy="0 0 0" />
       <limit lower="-1.5708" upper="1.5708" effort="1" velocity="1"/>
-      <axis xyz="1 0 0" />
+      <axis xyz="0 1 0" />
     </joint>
     <xacro:leg_transmission leg_number="${leg_number}" joint_number="2" />
@@ -105,5 +119,5 @@
   <!-- Assemble Body -->
   <xacro:macro name="millihex_body" params="">
-    <xacro:millihex_torso />
+    <xacro:millihex_torso color="Orange" />
     <xacro:millihex_leg leg_number="1" />
     <joint name="leg1_joint1" type="fixed">

Commit message: Added colors to Gazebo sim and updated axis rotations for joint controller

File: robot/millihex.xacro (robot description, xacro)
@@ -13,4 +13,11 @@
 	<xacro:property name="foot_mu1" value="10.0" />
   <xacro:property name="foot_mu2" value="10.0" />
+  <!-- Colors -->
+  <material name="Black">
+    <color rgba="0 0 0 1"/>
+  </material>
+  <material name="Orange">
+    <color rgba="0.945 0.35 0.133 1"/>
+  </material>
   <!-- Calculate Moment of Inertia of Box -->
   <xacro:macro name="box_inertia" params="mass x y z">
@@ -40,4 +47,5 @@
           <box size="${torso_x} ${torso_y} ${pcb_thickness_z}" />
         </geometry>
+        <material name="${color}"/>
       </visual>
     </link>
@@ -73,4 +81,5 @@
           <box size="${x_length} ${y_length} ${pcb_thickness_z}" />
         </geometry>
+        <material name="${color}"/>
       </visual>
     </link>
@@ -111,5 +120,5 @@
       <origin xyz="0 -${leg_link_y} 0" rpy="0 0 0" />
       <limit lower="-1.5708" upper="1.5708" effort="1" velocity="1"/>
-      <axis xyz="0 1 0" />
+      <axis xyz="1 0 0" />
     </joint>
     <xacro:leg_transmission leg_number="${leg_number}" joint_number="2" />

Commit message: Tuning effort and velocity params for link joint position controller

File: robot/millihex.xacro (robot description, xacro)
@@ -18,5 +18,5 @@
   </material>
   <material name="Orange">
-    <color rgba="0.945 0.35 0.133 1"/>
+    <color rgba="0.98 0.41 0.055 1"/>
   </material>
   <!-- Calculate Moment of Inertia of Box -->
@@ -119,5 +119,5 @@
       <child link="leg${leg_number}_link2" />
       <origin xyz="0 -${leg_link_y} 0" rpy="0 0 0" />
-      <limit lower="-1.5708" upper="1.5708" effort="1" velocity="1"/>
+      <limit lower="-1.5708" upper="1.5708" effort="0.01" velocity="0.0001"/>
       <axis xyz="1 0 0" />
     </joint>

Commit message: Changed friction properties foot_mu1 and foot_mu2

File: robot/millihex.xacro (robot description, xacro)
@@ -11,6 +11,6 @@
 	<xacro:property name="foot_kp" value="1000.0" />
 	<xacro:property name="foot_kd" value="1000.0" />
-	<xacro:property name="foot_mu1" value="10.0" />
-  <xacro:property name="foot_mu2" value="10.0" />
+	<xacro:property name="foot_mu1" value="0.2" />
+  <xacro:property name="foot_mu2" value="0.2" />
   <!-- Colors -->
   <material name="Black">

Commit message: Added link 3

File: robot/millihex.xacro (robot description, xacro)
@@ -124,4 +124,15 @@
     <xacro:leg_transmission leg_number="${leg_number}" joint_number="2" />
     <!-- TODO: link 3, horizontally oriented -->
+    <xacro:millihex_leg_link leg_number="${leg_number}" link_number="3"
+                             x_length="${leg_link_x}" y_length="${leg_link_y}"
+                             color="Black" />
+    <joint name="leg${leg_number}_joint3" type="revolute">
+      <parent link="leg${leg_number}_link2" />
+      <child link="leg${leg_number}_link3" />
+      <origin xyz="0 -${leg_link_y} 0" rpy="0 0 0" />
+      <limit lower="-1.5708" upper="1.5708" effort="0.01" velocity="0.0001"/>
+      <axis xyz="1 0 0" />
+    </joint>
+    <xacro:leg_transmission leg_number="${leg_number}" joint_number="2" />
     <!-- TODO: link 4, horizontally oriented -->
   </xacro:macro>

Commit message: Updated torso and leg masses

File: robot/millihex.xacro (robot description, xacro)
@@ -2,8 +2,8 @@
 <robot xmlns:xacro="http://www.ros.org/wiki/xacro" name="millihex">
   <!-- Properties -->
-  <xacro:property name="torso_mass" value="0.01" />
+  <xacro:property name="torso_mass" value="0.013" />
   <xacro:property name="torso_x" value="0.14" />
   <xacro:property name="torso_y" value="0.04" />
-  <xacro:property name="leg_link_mass" value="0.0008" />
+  <xacro:property name="leg_link_mass" value="0.00073" />
   <xacro:property name="leg_link_x" value="0.02" />
   <xacro:property name="leg_link_y" value="0.03" />

Commit message: FINAL MASS UPDATES

File: robot/millihex.xacro (robot description, xacro)
@@ -2,8 +2,8 @@
 <robot xmlns:xacro="http://www.ros.org/wiki/xacro" name="millihex">
   <!-- Properties -->
-  <xacro:property name="torso_mass" value="0.013" />
+  <xacro:property name="torso_mass" value="0.01" />
   <xacro:property name="torso_x" value="0.14" />
   <xacro:property name="torso_y" value="0.04" />
-  <xacro:property name="leg_link_mass" value="0.00073" />
+  <xacro:property name="leg_link_mass" value="0.0008" />
   <xacro:property name="leg_link_x" value="0.02" />
   <xacro:property name="leg_link_y" value="0.03" />

Commit message: Changed leg frictions from 0.2 to 0.5:

File: robot/millihex.xacro (robot description, xacro)
@@ -11,6 +11,6 @@
 	<xacro:property name="foot_kp" value="1000.0" />
 	<xacro:property name="foot_kd" value="1000.0" />
-	<xacro:property name="foot_mu1" value="0.2" />
-  <xacro:property name="foot_mu2" value="0.2" />
+	<xacro:property name="foot_mu1" value="0.5" />
+  <xacro:property name="foot_mu2" value="0.5" />
   <!-- Colors -->
   <material name="Black">

Commit message: Fixed robot leg link origin for collision tag to be identical to visual tag

File: robot/millihex.xacro (robot description, xacro)
@@ -71,5 +71,5 @@
       </inertial>
       <collision>
-        <origin xyz="0 0 ${pcb_thickness_z / 2}" rpy="0 0 0"/>
+        <origin xyz="-${x_length / 2} -${y_length / 2} 0" rpy="0 0 0"/>
         <geometry>
           <box size="${x_length} ${y_length} ${pcb_thickness_z}" />
