Commit message: Added comments and fixed indentation to make code easier to read

File: robot/millihex.xacro (robot description, xacro)
@@ -1,160 +1,155 @@
 <?xml version="1.0"?>
 <robot xmlns:xacro="http://www.ros.org/wiki/xacro" name="millihex">
-  <!-- Properties -->
-  <xacro:property name="torso_mass" value="0.01" />
-  <xacro:property name="torso_x" value="0.14" />
-  <xacro:property name="torso_y" value="0.04" />
-  <xacro:property name="leg_link_mass" value="0.0008" />
-  <xacro:property name="leg_link_x" value="0.02" />
-  <xacro:property name="leg_link_y" value="0.03" />
-  <xacro:property name="pcb_thickness_z" value="0.0005" />
-	<xacro:property name="foot_kp" value="1000.0" />
-	<xacro:property name="foot_kd" value="1000.0" />
-	<xacro:property name="foot_mu1" value="0.5" />
-  <xacro:property name="foot_mu2" value="0.5" />
-  <!-- Colors -->
-  <material name="Black">
-    <color rgba="0 0 0 1"/>
-  </material>
-  <material name="Orange">
-    <color rgba="0.98 0.41 0.055 1"/>
-  </material>
-  <!-- Calculate Moment of Inertia of Box -->
-  <xacro:macro name="box_inertia" params="mass x y z">
-    <inertia ixx="${mass*(y*y+z*z)/12}" ixy = "0" ixz = "0"
-             iyy="${mass*(x*x+z*z)/12}" iyz = "0"
-             izz="${mass*(x*x+y*y)/12}" />
-  </xacro:macro>
-  <!-- Base and Torso Definition -->
-  <xacro:macro name="millihex_torso" params="color">
-    <link name="base_link">
-    </link>
-    <link name="torso">
-      <inertial>
-        <origin xyz="0 0 ${pcb_thickness_z / 2}" rpy="0 0 0" />
-        <mass value="${torso_mass}" />
-        <xacro:box_inertia mass="${torso_mass}" x="${torso_x}" y="${torso_y}" z="${pcb_thickness_z}" />
-      </inertial>
-      <collision>
-        <origin xyz="0 0 ${pcb_thickness_z / 2}" rpy="0 0 0"/>
-        <geometry>
-          <box size="${torso_x} ${torso_y} ${pcb_thickness_z}" />
-        </geometry>
-      </collision>
-      <visual>
-        <origin xyz="0 0 0" rpy="0 0 0" />
-        <geometry>
-          <box size="${torso_x} ${torso_y} ${pcb_thickness_z}" />
-        </geometry>
-        <material name="${color}"/>
-      </visual>
-    </link>
-    <gazebo reference="torso">
-      <kp>${foot_kp}</kp>
-      <kd>${foot_kd}</kd>
-      <mu1>${foot_mu1}</mu1>
-      <mu2>${foot_mu2}</mu2>
-      <material>Gazebo/${color}</material>
-    </gazebo>
-    <joint name="base_joint" type="fixed">
-        <parent link="base_link"/>
-        <child link="torso"/>
-    </joint>
-  </xacro:macro>
-  <!-- Leg Link Definition -->
-  <xacro:macro name="millihex_leg_link" params="leg_number link_number x_length y_length color">
-    <link name="leg${leg_number}_link${link_number}">
-      <inertial>
-        <origin xyz="0 0 ${pcb_thickness_z / 2}" rpy="0 0 0" />
-        <mass value="${leg_link_mass}" />
-        <xacro:box_inertia mass="${leg_link_mass}" x="${x_length}" y="${y_length}" z="${pcb_thickness_z}" />
-      </inertial>
-      <collision>
-        <origin xyz="-${x_length / 2} -${y_length / 2} 0" rpy="0 0 0"/>
-        <geometry>
-          <box size="${x_length} ${y_length} ${pcb_thickness_z}" />
-        </geometry>
-      </collision>
-      <visual>
-        <origin xyz="-${x_length / 2} -${y_length / 2} 0" rpy="0 0 0" />
-        <geometry>
-          <box size="${x_length} ${y_length} ${pcb_thickness_z}" />
-        </geometry>
-        <material name="${color}"/>
-      </visual>
-    </link>
-    <gazebo reference="leg${leg_number}_link${link_number}">
-      <kp>${foot_kp}</kp>
-      <kd>${foot_kd}</kd>
-      <mu1>${foot_mu1}</mu1>
-      <mu2>${foot_mu2}</mu2>
-      <material>Gazebo/${color}</material>
-    </gazebo>
-  </xacro:macro>
-  <!-- Leg Joint Transmission -->
-  <xacro:macro name="leg_transmission" params="leg_number joint_number">
-    <transmission name="leg${leg_number}_joint${joint_number}_tran">
-      <type>transmission_interface/SimpleTransmission</type>
-      <joint name="leg${leg_number}_joint${joint_number}">
-        <hardwareInterface>hardware_interface/EffortJointInterface</hardwareInterface>
-      </joint>
-      <actuator name="leg${leg_number}_joint${joint_number}_motor">
-        <hardwareInterface>EffortJointInterface</hardwareInterface>
-        <mechanicalReduction>1</mechanicalReduction>
-      </actuator>
-    </transmission>
-  </xacro:macro>
-  <!-- Assemble Leg -->
-  <xacro:macro name="millihex_leg" params="leg_number">
-    <!-- link 1 (shoulder link), horizontally oriented -->
-    <xacro:millihex_leg_link leg_number="${leg_number}" link_number="1"
-                             x_length="${leg_link_x}" y_length="${leg_link_y}"
-                             color="Black" />
-    <!-- link 2, vertically oriented -->
-    <xacro:millihex_leg_link leg_number="${leg_number}" link_number="2"
-                             x_length="${leg_link_y}" y_length="${leg_link_x}"
-                             color="Orange" />
-    <joint name="leg${leg_number}_joint2" type="revolute">
-      <parent link="leg${leg_number}_link1" />
-      <child link="leg${leg_number}_link2" />
-      <origin xyz="0 -${leg_link_y} 0" rpy="0 0 0" />
-      <limit lower="-1.5708" upper="1.5708" effort="0.01" velocity="0.0001"/>
-      <axis xyz="1 0 0" />
-    </joint>
-    <xacro:leg_transmission leg_number="${leg_number}" joint_number="2" />
-    <!-- TODO: link 3, horizontally oriented -->
-    <xacro:millihex_leg_link leg_number="${leg_number}" link_number="3"
-                             x_length="${leg_link_x}" y_length="${leg_link_y}"
-                             color="Black" />
-    <joint name="leg${leg_number}_joint3" type="revolute">
-      <parent link="leg${leg_number}_link2" />
-      <child link="leg${leg_number}_link3" />
-      <origin xyz="0 -${leg_link_y} 0" rpy="0 0 0" />
-      <limit lower="-1.5708" upper="1.5708" effort="0.01" velocity="0.0001"/>
-      <axis xyz="1 0 0" />
-    </joint>
-    <xacro:leg_transmission leg_number="${leg_number}" joint_number="2" />
-    <!-- TODO: link 4, horizontally oriented -->
-  </xacro:macro>
-  <!-- Assemble Body -->
-  <xacro:macro name="millihex_body" params="">
-    <xacro:millihex_torso color="Orange" />
-    <xacro:millihex_leg leg_number="1" />
-    <joint name="leg1_joint1" type="fixed">
-      <parent link="torso" />
-      <child link="leg1_link1" />
-      <origin xyz="${torso_x / 2} -${torso_y / 2} 0" rpy="0 0 0" />
-    </joint>
-  </xacro:macro>
-  <!-- Add Gazebo Control Library -->
-  <xacro:macro name="millihex_control" params="namespace">
-    <gazebo>
-      <plugin name="gazebo_ros_control" filename="libgazebo_ros_control.so">
-        <robotNamespace>/${namespace}</robotNamespace>
-      </plugin>
-    </gazebo>
-  </xacro:macro>
-  <!-- Build Robot by Filling in Macro Parameters -->
-  <xacro:millihex_body />
-  <xacro:millihex_control namespace="millihex" />
+    <!-- Physical Properties -->
+    <xacro:property name="torso_mass" value="0.01" />
+    <xacro:property name="torso_x" value="0.14" />
+    <xacro:property name="torso_y" value="0.04" />
+    <xacro:property name="leg_link_mass" value="0.0008" />
+    <xacro:property name="leg_link_x" value="0.02" />
+    <xacro:property name="leg_link_y" value="0.03" />
+    <xacro:property name="pcb_thickness_z" value="0.0005" />
+    <xacro:property name="foot_kp" value="1000.0" />
+    <xacro:property name="foot_kd" value="1000.0" />
+    <xacro:property name="foot_mu1" value="0.5" />
+    <xacro:property name="foot_mu2" value="0.5" />
+    <!-- Color Definitions -->
+    <material name="Black">
+        <color rgba="0 0 0 1"/>
+    </material>
+    <material name="Orange">
+        <color rgba="0.98 0.41 0.055 1"/>
+    </material>
+    <!-- Calculate Moment of Inertia of Box -->
+    <xacro:macro name="box_inertia" params="mass x y z">
+        <inertia ixx="${mass*(y*y+z*z)/12}" ixy = "0" ixz = "0"
+            iyy="${mass*(x*x+z*z)/12}" iyz = "0" izz="${mass*(x*x+y*y)/12}" />
+    </xacro:macro>
+    <!-- Base and Torso Definition -->
+    <xacro:macro name="millihex_torso" params="color">
+        <!-- Empty Base Link to attach robot to world -->
+        <link name="base_link">
+        </link>
+        <!-- Torso geometry without legs -->
+        <link name="torso">
+            <inertial>
+                <origin xyz="0 0 ${pcb_thickness_z / 2}" rpy="0 0 0" />
+                <mass value="${torso_mass}" />
+                <xacro:box_inertia mass="${torso_mass}" x="${torso_x}" y="${torso_y}" z="${pcb_thickness_z}" />
+            </inertial>
+            <collision>
+                <origin xyz="0 0 0" rpy="0 0 0"/>
+                <geometry>
+                    <box size="${torso_x} ${torso_y} ${pcb_thickness_z}" />
+                </geometry>
+            </collision>
+            <visual>
+                <origin xyz="0 0 0" rpy="0 0 0" />
+                <geometry>
+                    <box size="${torso_x} ${torso_y} ${pcb_thickness_z}" />
+                </geometry>
+                <material name="${color}"/>
+            </visual>
+        </link>
+        <!-- Gazebo properties -->
+        <gazebo reference="torso">
+            <kp>${foot_kp}</kp>
+            <kd>${foot_kd}</kd>
+            <mu1>${foot_mu1}</mu1>
+            <mu2>${foot_mu2}</mu2>
+            <material>Gazebo/${color}</material>
+        </gazebo>
+        <!-- Join Base Link and Torso -->
+        <joint name="base_joint" type="fixed">
+            <parent link="base_link"/>
+            <child link="torso"/>
+        </joint>
+    </xacro:macro>
+    <!-- Leg Link Definition -->
+    <xacro:macro name="millihex_leg_link" params="leg_number link_number x_length y_length color">
+        <!-- Leg geometry -->
+        <link name="leg${leg_number}_link${link_number}">
+            <inertial>
+                <origin xyz="0 0 ${pcb_thickness_z / 2}" rpy="0 0 0" />
+                <mass value="${leg_link_mass}" />
+                <xacro:box_inertia mass="${leg_link_mass}" x="${x_length}" y="${y_length}" z="${pcb_thickness_z}" />
+            </inertial>
+            <collision>
+                <origin xyz="-${x_length / 2} -${y_length / 2} 0" rpy="0 0 0"/>
+                <geometry>
+                    <box size="${x_length} ${y_length} ${pcb_thickness_z}" />
+                </geometry>
+            </collision>
+            <visual>
+                <origin xyz="-${x_length / 2} -${y_length / 2} 0" rpy="0 0 0" />
+                <geometry>
+                    <box size="${x_length} ${y_length} ${pcb_thickness_z}" />
+                </geometry>
+                <material name="${color}"/>
+            </visual>
+        </link>
+        <!-- Gazebo properties -->
+        <gazebo reference="leg${leg_number}_link${link_number}">
+            <kp>${foot_kp}</kp>
+            <kd>${foot_kd}</kd>
+            <mu1>${foot_mu1}</mu1>
+            <mu2>${foot_mu2}</mu2>
+            <material>Gazebo/${color}</material>
+        </gazebo>
+    </xacro:macro>
+    <!-- Leg Joint Transmission -->
+    <xacro:macro name="leg_transmission" params="leg_number joint_number">
+        <transmission name="leg${leg_number}_joint${joint_number}_tran">
+            <type>transmission_interface/SimpleTransmission</type>
+            <joint name="leg${leg_number}_joint${joint_number}">
+                <hardwareInterface>hardware_interface/EffortJointInterface</hardwareInterface>
+            </joint>
+            <actuator name="leg${leg_number}_joint${joint_number}_motor">
+                <hardwareInterface>EffortJointInterface</hardwareInterface>
+                <mechanicalReduction>1</mechanicalReduction>
+            </actuator>
+        </transmission>
+    </xacro:macro>
+    <!-- Assemble Leg -->
+    <xacro:macro name="millihex_leg" params="leg_number">
+        <!-- Link 1 (shoulder link), horizontally oriented -->
+        <xacro:millihex_leg_link leg_number="${leg_number}" link_number="1"
+            x_length="${leg_link_x}" y_length="${leg_link_y}" color="Black" />
+        <!-- Link 2, vertically oriented -->
+        <xacro:millihex_leg_link leg_number="${leg_number}" link_number="2"
+            x_length="${leg_link_y}" y_length="${leg_link_x}" color="Orange" />
+        <joint name="leg${leg_number}_joint2" type="revolute">
+            <parent link="leg${leg_number}_link1" />
+            <child link="leg${leg_number}_link2" />
+            <origin xyz="0 -${leg_link_y} 0" rpy="0 0 0" />
+            <limit lower="-1.5708" upper="1.5708" effort="0.01" velocity="0.0001"/>
+            <axis xyz="1 0 0" />
+        </joint>
+        <xacro:leg_transmission leg_number="${leg_number}" joint_number="2" />
+        <!-- TODO: Link 3, horizontally oriented -->
+        <!-- TODO: Link 4, horizontally oriented -->
+    </xacro:macro>
+    <!-- Assemble Body -->
+    <xacro:macro name="millihex_body" params="">
+        <!-- Call Torso xacro -->
+        <xacro:millihex_torso color="Orange" />
+        <!-- Define Leg 1-->
+        <xacro:millihex_leg leg_number="1" />
+        <!-- Joint 1, Leg1 Link1-->
+        <joint name="leg1_joint1" type="fixed">
+            <parent link="torso" />
+            <child link="leg1_link1" />
+            <origin xyz="${torso_x / 2} -${torso_y / 2} 0" rpy="0 0 0" />
+        </joint>
+    </xacro:macro>
+    <!-- Add Gazebo Control Library -->
+    <xacro:macro name="millihex_control" params="namespace">
+        <gazebo>
+            <plugin name="gazebo_ros_control" filename="libgazebo_ros_control.so">
+                <robotNamespace>/${namespace}</robotNamespace>
+            </plugin>
+        </gazebo>
+    </xacro:macro>
+    <!-- Build Robot by Filling in Macro Parameters -->
+    <xacro:millihex_body />
+    <xacro:millihex_control namespace="millihex" />
 </robot>

Commit message: Changed tab formatting

File: robot/millihex.xacro (robot description, xacro)
@@ -43,5 +43,5 @@
       </collision>
       <visual>
-        <origin xyz="0 0 0" rpy="0 0 0" />
+        <origin xyz="0 0 ${pcb_thickness_z / 2}" rpy="0 0 0" />
         <geometry>
           <box size="${torso_x} ${torso_y} ${pcb_thickness_z}" />
@@ -124,15 +124,4 @@
     <xacro:leg_transmission leg_number="${leg_number}" joint_number="2" />
     <!-- TODO: link 3, horizontally oriented -->
-    <xacro:millihex_leg_link leg_number="${leg_number}" link_number="3"
-                             x_length="${leg_link_x}" y_length="${leg_link_y}"
-                             color="Black" />
-    <joint name="leg${leg_number}_joint3" type="revolute">
-      <parent link="leg${leg_number}_link2" />
-      <child link="leg${leg_number}_link3" />
-      <origin xyz="0 -${leg_link_y} 0" rpy="0 0 0" />
-      <limit lower="-1.5708" upper="1.5708" effort="0.01" velocity="0.0001"/>
-      <axis xyz="1 0 0" />
-    </joint>
-    <xacro:leg_transmission leg_number="${leg_number}" joint_number="2" />
     <!-- TODO: link 4, horizontally oriented -->
   </xacro:macro>

Commit message: Added Leg Link 3 to a leg

File: robot/millihex.xacro (robot description, xacro)
@@ -126,5 +126,15 @@
         </joint>
         <xacro:leg_transmission leg_number="${leg_number}" joint_number="2" />
-        <!-- TODO: Link 3, horizontally oriented -->
+        <!-- Link 3, horizontally oriented -->
+        <xacro:millihex_leg_link leg_number="${leg_number}" link_number="3"
+            x_length="${leg_link_x}" y_length="${leg_link_y}" color="Black" />
+        <joint name="leg${leg_number}_joint3" type="revolute">
+            <parent link="leg${leg_number}_link2" />
+            <child link="leg${leg_number}_link3" />
+            <origin xyz="-${leg_link_y} 0 0" rpy="0 0 0" />
+            <limit lower="-1.5708" upper="1.5708" effort="0.01" velocity="0.0001"/>
+            <axis xyz="0 1 0" />
+        </joint>
+        <xacro:leg_transmission leg_number="${leg_number}" joint_number="3" />
         <!-- TODO: Link 4, horizontally oriented -->
     </xacro:macro>

Commit message: Added Leg Link 4 to leg

File: robot/millihex.xacro (robot description, xacro)
@@ -137,5 +137,15 @@
         </joint>
         <xacro:leg_transmission leg_number="${leg_number}" joint_number="3" />
-        <!-- TODO: Link 4, horizontally oriented -->
+        <!-- Link 4, horizontally oriented -->
+        <xacro:millihex_leg_link leg_number="${leg_number}" link_number="4"
+            x_length="${leg_link_x}" y_length="${leg_link_y}" color="Orange" />
+        <joint name="leg${leg_number}_joint4" type="revolute">
+            <parent link="leg${leg_number}_link3" />
+            <child link="leg${leg_number}_link4" />
+            <origin xyz="0 -${leg_link_y} 0" rpy="0 0 0" />
+            <limit lower="-1.5708" upper="1.5708" effort="0.01" velocity="0.0001"/>
+            <axis xyz="1 0 0" />
+        </joint>
+        <xacro:leg_transmission leg_number="${leg_number}" joint_number="4" />
     </xacro:macro>
     <!-- Assemble Body -->

Commit message: Added Leg2

File: robot/millihex.xacro (robot description, xacro)
@@ -153,7 +153,7 @@
         <!-- Call Torso xacro -->
         <xacro:millihex_torso color="Orange" />
-        <!-- Define Leg 1-->
+        <!-- Leg 1-->
         <xacro:millihex_leg leg_number="1" />
-        <!-- Joint 1, Leg1 Link1-->
+        <!-- Joint 1 -->
         <joint name="leg1_joint1" type="fixed">
             <parent link="torso" />
@@ -161,4 +161,20 @@
             <origin xyz="${torso_x / 2} -${torso_y / 2} 0" rpy="0 0 0" />
         </joint>
+        <!-- Leg 2 -->
+        <xacro:millihex_leg leg_number="2" />
+        <!-- Leg 2, Joint 1 -->
+        <joint name="leg2_joint1" type="fixed">
+            <parent link="torso" />
+            <child link="leg2_link1" />
+            <origin xyz="${leg_link_x / 2} -${torso_y / 2} 0" rpy="0 0 0" />
+        </joint>
+        <!-- Leg 3 -->
+        <!-- Leg 3, Joint 1 -->
+        <!-- Leg 4 -->
+        <!-- Leg 4, Joint 1 -->
+        <!-- Leg 5 -->
+        <!-- Leg 5, Joint 1 -->
+        <!-- Leg 6 -->
+        <!-- Leg 6, Joint 1 -->
     </xacro:macro>
     <!-- Add Gazebo Control Library -->
