Commit message: Renamed leg joint and link indices to start from 0

File: robot/millihex.xacro (robot description, xacro)
@@ -112,40 +112,40 @@
     <!-- Assemble Leg -->
     <xacro:macro name="millihex_leg" params="leg_number">
-        <!-- Link 1 (shoulder link), horizontally oriented -->
+        <!-- Link 0 (shoulder link), horizontally oriented -->
+        <xacro:millihex_leg_link leg_number="${leg_number}" link_number="0"
+            x_length="${leg_link_x}" y_length="${leg_link_y}" color="Black" />
+        <!-- Link 1, vertically oriented -->
         <xacro:millihex_leg_link leg_number="${leg_number}" link_number="1"
-            x_length="${leg_link_x}" y_length="${leg_link_y}" color="Black" />
-        <!-- Link 2, vertically oriented -->
-        <xacro:millihex_leg_link leg_number="${leg_number}" link_number="2"
             x_length="${leg_link_y}" y_length="${leg_link_x}" color="Orange" />
-        <joint name="leg${leg_number}_joint2" type="revolute">
-            <parent link="leg${leg_number}_link1" />
-            <child link="leg${leg_number}_link2" />
+        <joint name="leg${leg_number}_joint1" type="revolute">
+            <parent link="leg${leg_number}_link0" />
+            <child link="leg${leg_number}_link1" />
             <origin xyz="0 -${leg_link_y} 0" rpy="0 0 0" />
             <limit lower="-1.5708" upper="1.5708" effort="0.01" velocity="0.0001"/>
             <axis xyz="1 0 0" />
         </joint>
-        <xacro:leg_transmission leg_number="${leg_number}" joint_number="2" />
-        <!-- Link 3, horizontally oriented -->
-        <xacro:millihex_leg_link leg_number="${leg_number}" link_number="3"
+        <xacro:leg_transmission leg_number="${leg_number}" joint_number="1" />
+        <!-- Link 2, horizontally oriented -->
+        <xacro:millihex_leg_link leg_number="${leg_number}" link_number="2"
             x_length="${leg_link_x}" y_length="${leg_link_y}" color="Black" />
-        <joint name="leg${leg_number}_joint3" type="revolute">
-            <parent link="leg${leg_number}_link2" />
-            <child link="leg${leg_number}_link3" />
+        <joint name="leg${leg_number}_joint2" type="revolute">
+            <parent link="leg${leg_number}_link1" />
+            <child link="leg${leg_number}_link2" />
             <origin xyz="-${leg_link_y} 0 0" rpy="0 0 0" />
             <limit lower="-1.5708" upper="1.5708" effort="0.01" velocity="0.0001"/>
             <axis xyz="0 1 0" />
         </joint>
-        <xacro:leg_transmission leg_number="${leg_number}" joint_number="3" />
-        <!-- Link 4, horizontally oriented -->
-        <xacro:millihex_leg_link leg_number="${leg_number}" link_number="4"
+        <xacro:leg_transmission leg_number="${leg_number}" joint_number="2" />
+        <!-- Link 3, horizontally oriented -->
+        <xacro:millihex_leg_link leg_number="${leg_number}" link_number="3"
             x_length="${leg_link_x}" y_length="${leg_link_y}" color="Orange" />
-        <joint name="leg${leg_number}_joint4" type="revolute">
-            <parent link="leg${leg_number}_link3" />
-            <child link="leg${leg_number}_link4" />
+        <joint name="leg${leg_number}_joint3" type="revolute">
+            <parent link="leg${leg_number}_link2" />
+            <child link="leg${leg_number}_link3" />
             <origin xyz="0 -${leg_link_y} 0" rpy="0 0 0" />
             <limit lower="-1.5708" upper="1.5708" effort="0.01" velocity="0.0001"/>
             <axis xyz="1 0 0" />
         </joint>
-        <xacro:leg_transmission leg_number="${leg_number}" joint_number="4" />
+        <xacro:leg_transmission leg_number="${leg_number}" joint_number="3" />
     </xacro:macro>
     <!-- Assemble Body -->
@@ -155,26 +155,26 @@
         <!-- Leg 1-->
         <xacro:millihex_leg leg_number="1" />
-        <!-- Joint 1 -->
-        <joint name="leg1_joint1" type="fixed">
+        <!-- Leg 1, Joint 0 (fixed, shoulder joint)-->
+        <joint name="leg1_joint0" type="fixed">
             <parent link="torso" />
-            <child link="leg1_link1" />
+            <child link="leg1_link0" />
             <origin xyz="${torso_x / 2} -${torso_y / 2} 0" rpy="0 0 0" />
         </joint>
         <!-- Leg 2 -->
         <xacro:millihex_leg leg_number="2" />
-        <!-- Leg 2, Joint 1 -->
-        <joint name="leg2_joint1" type="fixed">
+        <!-- Leg 2, Joint 0 (fixed, shoulder joint) -->
+        <joint name="leg2_joint0" type="fixed">
             <parent link="torso" />
-            <child link="leg2_link1" />
+            <child link="leg2_link0" />
             <origin xyz="${leg_link_x / 2} -${torso_y / 2} 0" rpy="0 0 0" />
         </joint>
         <!-- Leg 3 -->
-        <!-- Leg 3, Joint 1 -->
+        <!-- Leg 3, Joint 0 (fixed, shoulder joint) -->
         <!-- Leg 4 -->
-        <!-- Leg 4, Joint 1 -->
+        <!-- Leg 4, Joint 0 (fixed, shoulder joint) -->
         <!-- Leg 5 -->
-        <!-- Leg 5, Joint 1 -->
+        <!-- Leg 5, Joint 0 (fixed, shoulder joint) -->
         <!-- Leg 6 -->
-        <!-- Leg 6, Joint 1 -->
+        <!-- Leg 6, Joint 0 (fixed, shoulder joint) -->
     </xacro:macro>
     <!-- Add Gazebo Control Library -->

Commit message: Added Leg 3

File: robot/millihex.xacro (robot description, xacro)
@@ -170,5 +170,11 @@
         </joint>
         <!-- Leg 3 -->
+        <xacro:millihex_leg leg_number="3" />
         <!-- Leg 3, Joint 0 (fixed, shoulder joint) -->
+        <joint name="leg3_joint0" type="fixed">
+            <parent link="torso" />
+            <child link="leg3_link0" />
+            <origin xyz="-${torso_x / 2 - leg_link_x} -${torso_y / 2} 0" rpy="0 0 0" />
+        </joint>
         <!-- Leg 4 -->
         <!-- Leg 4, Joint 0 (fixed, shoulder joint) -->

Commit message: Added Leg 4

File: robot/millihex.xacro (robot description, xacro)
@@ -178,5 +178,11 @@
         </joint>
         <!-- Leg 4 -->
+        <xacro:millihex_leg leg_number="4" />
         <!-- Leg 4, Joint 0 (fixed, shoulder joint) -->
+        <joint name="leg4_joint0" type="fixed">
+            <parent link="torso" />
+            <child link="leg4_link0" />
+            <origin xyz="${torso_x / 2} ${torso_y / 2} 0" rpy="3.1416 0 0" />
+        </joint>
         <!-- Leg 5 -->
         <!-- Leg 5, Joint 0 (fixed, shoulder joint) -->

Commit message: Added Leg 5 and its joit position controllers

File: robot/millihex.xacro (robot description, xacro)
@@ -186,5 +186,11 @@
         </joint>
         <!-- Leg 5 -->
+        <xacro:millihex_leg leg_number="5" />
         <!-- Leg 5, Joint 0 (fixed, shoulder joint) -->
+        <joint name="leg5_joint0" type="fixed">
+            <parent link="torso" />
+            <child link="leg5_link0" />
+            <origin xyz="${leg_link_x / 2} ${torso_y / 2} 0" rpy="3.1416 0 0" />
+        </joint>
         <!-- Leg 6 -->
         <!-- Leg 6, Joint 0 (fixed, shoulder joint) -->

Commit message: Added Leg 6 and corresponding joint position controllers

File: robot/millihex.xacro (robot description, xacro)
@@ -194,5 +194,11 @@
         </joint>
         <!-- Leg 6 -->
+        <xacro:millihex_leg leg_number="6" />
         <!-- Leg 6, Joint 0 (fixed, shoulder joint) -->
+        <joint name="leg6_joint0" type="fixed">
+            <parent link="torso" />
+            <child link="leg6_link0" />
+            <origin xyz="-${torso_x / 2 - leg_link_x} ${torso_y / 2} 0" rpy="3.1416 0 0" />
+        </joint>
     </xacro:macro>
     <!-- Add Gazebo Control Library -->

Commit message: Added joint_limit, joint_effort, and joint_velocity property macros to easily test different joint values

File: robot/millihex.xacro (robot description, xacro)
@@ -8,4 +8,7 @@
     <xacro:property name="leg_link_x" value="0.02" />
     <xacro:property name="leg_link_y" value="0.03" />
+    <xacro:property name="joint_limit" value="1.5708" />
+    <xacro:property name="joint_effort" value="0.01" />
+    <xacro:property name="joint_velocity" value="0.0001" />
     <xacro:property name="pcb_thickness_z" value="0.0005" />
     <xacro:property name="foot_kp" value="1000.0" />
@@ -20,5 +23,5 @@
         <color rgba="0.98 0.41 0.055 1"/>
     </material>
-    <!-- Calculate Moment of Inertia of Box -->
+    <!-- Calculate Moment of Inertia of a Box -->
     <xacro:macro name="box_inertia" params="mass x y z">
         <inertia ixx="${mass*(y*y+z*z)/12}" ixy = "0" ixz = "0"
@@ -35,5 +38,6 @@
                 <origin xyz="0 0 ${pcb_thickness_z / 2}" rpy="0 0 0" />
                 <mass value="${torso_mass}" />
-                <xacro:box_inertia mass="${torso_mass}" x="${torso_x}" y="${torso_y}" z="${pcb_thickness_z}" />
+                <xacro:box_inertia mass="${torso_mass}" x="${torso_x}"
+                    y="${torso_y}" z="${pcb_thickness_z}" />
             </inertial>
             <collision>
@@ -66,5 +70,6 @@
     </xacro:macro>
     <!-- Leg Link Definition -->
-    <xacro:macro name="millihex_leg_link" params="leg_number link_number x_length y_length color">
+    <xacro:macro name="millihex_leg_link"
+        params="leg_number link_number x_length y_length color">
         <!-- Leg geometry -->
         <link name="leg${leg_number}_link${link_number}">
@@ -72,5 +77,6 @@
                 <origin xyz="0 0 ${pcb_thickness_z / 2}" rpy="0 0 0" />
                 <mass value="${leg_link_mass}" />
-                <xacro:box_inertia mass="${leg_link_mass}" x="${x_length}" y="${y_length}" z="${pcb_thickness_z}" />
+                <xacro:box_inertia mass="${leg_link_mass}" x="${x_length}"
+                    y="${y_length}" z="${pcb_thickness_z}" />
             </inertial>
             <collision>
@@ -102,5 +108,7 @@
             <type>transmission_interface/SimpleTransmission</type>
             <joint name="leg${leg_number}_joint${joint_number}">
-                <hardwareInterface>hardware_interface/EffortJointInterface</hardwareInterface>
+                <hardwareInterface>
+                    hardware_interface/EffortJointInterface
+                </hardwareInterface>
             </joint>
             <actuator name="leg${leg_number}_joint${joint_number}_motor">
@@ -122,5 +130,6 @@
             <child link="leg${leg_number}_link1" />
             <origin xyz="0 -${leg_link_y} 0" rpy="0 0 0" />
-            <limit lower="-1.5708" upper="1.5708" effort="0.01" velocity="0.0001"/>
+            <limit lower="-${joint_limit}" upper="${joint_limit}"
+                effort="${joint_effort}" velocity="${joint_velocity}"/>
             <axis xyz="1 0 0" />
         </joint>
@@ -133,5 +142,6 @@
             <child link="leg${leg_number}_link2" />
             <origin xyz="-${leg_link_y} 0 0" rpy="0 0 0" />
-            <limit lower="-1.5708" upper="1.5708" effort="0.01" velocity="0.0001"/>
+            <limit lower="-${joint_limit}" upper="${joint_limit}"
+                effort="${joint_effort}" velocity="${joint_velocity}"/>
             <axis xyz="0 1 0" />
         </joint>
@@ -144,5 +154,6 @@
             <child link="leg${leg_number}_link3" />
             <origin xyz="0 -${leg_link_y} 0" rpy="0 0 0" />
-            <limit lower="-1.5708" upper="1.5708" effort="0.01" velocity="0.0001"/>
+            <limit lower="-${joint_limit}" upper="${joint_limit}"
+                effort="${joint_effort}" velocity="${joint_velocity}"/>
             <axis xyz="1 0 0" />
         </joint>
@@ -175,5 +186,6 @@
             <parent link="torso" />
             <child link="leg3_link0" />
-            <origin xyz="-${torso_x / 2 - leg_link_x} -${torso_y / 2} 0" rpy="0 0 0" />
+            <origin xyz="-${torso_x / 2 - leg_link_x} -${torso_y / 2} 0"
+                rpy="0 0 0" />
         </joint>
         <!-- Leg 4 -->
@@ -199,5 +211,6 @@
             <parent link="torso" />
             <child link="leg6_link0" />
-            <origin xyz="-${torso_x / 2 - leg_link_x} ${torso_y / 2} 0" rpy="3.1416 0 0" />
+            <origin xyz="-${torso_x / 2 - leg_link_x} ${torso_y / 2} 0"
+                rpy="3.1416 0 0" />
         </joint>
     </xacro:macro>

Commit message: Added damping and friction property variables to xacro

File: robot/millihex.xacro (robot description, xacro)
@@ -10,16 +10,18 @@
     <xacro:property name="joint_limit" value="1.5708" />
     <xacro:property name="joint_effort" value="0.01" />
-    <xacro:property name="joint_velocity" value="0.0001" />
+    <xacro:property name="joint_velocity" value="0.01" />
     <xacro:property name="pcb_thickness_z" value="0.0005" />
     <xacro:property name="foot_kp" value="1000.0" />
-    <xacro:property name="foot_kd" value="1000.0" />
+    <xacro:property name="foot_kd" value="1.0" />
     <xacro:property name="foot_mu1" value="0.5" />
     <xacro:property name="foot_mu2" value="0.5" />
+    <xacro:property name="joint_damping" value="" />
+    <xacro:property name="joint_friction" value="" />
     <!-- Color Definitions -->
     <material name="Black">
-        <color rgba="0 0 0 1"/>
+        <color rgba="0 0 0 1" />
     </material>
     <material name="Orange">
-        <color rgba="0.98 0.41 0.055 1"/>
+        <color rgba="0.98 0.41 0.055 1" />
     </material>
     <!-- Calculate Moment of Inertia of a Box -->
@@ -42,5 +44,5 @@
             </inertial>
             <collision>
-                <origin xyz="0 0 0" rpy="0 0 0"/>
+                <origin xyz="0 0 0" rpy="0 0 0" />
                 <geometry>
                     <box size="${torso_x} ${torso_y} ${pcb_thickness_z}" />
@@ -52,5 +54,5 @@
                     <box size="${torso_x} ${torso_y} ${pcb_thickness_z}" />
                 </geometry>
-                <material name="${color}"/>
+                <material name="${color}" />
             </visual>
         </link>
@@ -65,6 +67,6 @@
         <!-- Join Base Link and Torso -->
         <joint name="base_joint" type="fixed">
-            <parent link="base_link"/>
-            <child link="torso"/>
+            <parent link="base_link" />
+            <child link="torso" />
         </joint>
     </xacro:macro>
@@ -81,5 +83,5 @@
             </inertial>
             <collision>
-                <origin xyz="-${x_length / 2} -${y_length / 2} 0" rpy="0 0 0"/>
+                <origin xyz="-${x_length / 2} -${y_length / 2} 0" rpy="0 0 0" />
                 <geometry>
                     <box size="${x_length} ${y_length} ${pcb_thickness_z}" />
@@ -113,6 +115,8 @@
             </joint>
             <actuator name="leg${leg_number}_joint${joint_number}_motor">
-                <hardwareInterface>EffortJointInterface</hardwareInterface>
-                <mechanicalReduction>1</mechanicalReduction>
+                <hardwareInterface>
+                    hardware_interface/EffortJointInterface
+                </hardwareInterface>
+                <mechanicalReduction>50</mechanicalReduction>
             </actuator>
         </transmission>
@@ -131,5 +135,5 @@
             <origin xyz="0 -${leg_link_y} 0" rpy="0 0 0" />
             <limit lower="-${joint_limit}" upper="${joint_limit}"
-                effort="${joint_effort}" velocity="${joint_velocity}"/>
+                effort="${joint_effort}" velocity="${joint_velocity}" />
             <axis xyz="1 0 0" />
         </joint>
@@ -143,5 +147,5 @@
             <origin xyz="-${leg_link_y} 0 0" rpy="0 0 0" />
             <limit lower="-${joint_limit}" upper="${joint_limit}"
-                effort="${joint_effort}" velocity="${joint_velocity}"/>
+                effort="${joint_effort}" velocity="${joint_velocity}" />
             <axis xyz="0 1 0" />
         </joint>
@@ -155,5 +159,5 @@
             <origin xyz="0 -${leg_link_y} 0" rpy="0 0 0" />
             <limit lower="-${joint_limit}" upper="${joint_limit}"
-                effort="${joint_effort}" velocity="${joint_velocity}"/>
+                effort="${joint_effort}" velocity="${joint_velocity}" />
             <axis xyz="1 0 0" />
         </joint>

Commit message: Changed joint limit variable names to be more explicit that they are not controlling the position, effort, and velocity themselves but only setting a boundary/limit on them

File: robot/millihex.xacro (robot description, xacro)
@@ -8,7 +8,8 @@
     <xacro:property name="leg_link_x" value="0.02" />
     <xacro:property name="leg_link_y" value="0.03" />
-    <xacro:property name="joint_limit" value="1.5708" />
-    <xacro:property name="joint_effort" value="0.01" />
-    <xacro:property name="joint_velocity" value="0.01" />
+    <xacro:property name="joint_upper_limit" value="1.5708" />
+    <xacro:property name="joint_lower_limit" value="-1.5708" />
+    <xacro:property name="joint_effort_limit" value="0.01" />
+    <xacro:property name="joint_velocity_limit" value="0.01" />
     <xacro:property name="pcb_thickness_z" value="0.0005" />
     <xacro:property name="foot_kp" value="1000.0" />
@@ -118,5 +119,5 @@
                     hardware_interface/EffortJointInterface
                 </hardwareInterface>
-                <mechanicalReduction>50</mechanicalReduction>
+                <mechanicalReduction>1</mechanicalReduction>
             </actuator>
         </transmission>
@@ -134,6 +135,8 @@
             <child link="leg${leg_number}_link1" />
             <origin xyz="0 -${leg_link_y} 0" rpy="0 0 0" />
-            <limit lower="-${joint_limit}" upper="${joint_limit}"
-                effort="${joint_effort}" velocity="${joint_velocity}" />
+            <limit lower="${joint_lower_limit}"
+                   upper="${joint_upper_limit}"
+                   effort="${joint_effort_limit}"
+                   velocity="${joint_velocity_limit}" />
             <axis xyz="1 0 0" />
         </joint>
@@ -146,6 +149,8 @@
             <child link="leg${leg_number}_link2" />
             <origin xyz="-${leg_link_y} 0 0" rpy="0 0 0" />
-            <limit lower="-${joint_limit}" upper="${joint_limit}"
-                effort="${joint_effort}" velocity="${joint_velocity}" />
+            <limit lower="${joint_lower_limit}"
+                   upper="${joint_upper_limit}"
+                   effort="${joint_effort_limit}"
+                   velocity="${joint_velocity_limit}" />
             <axis xyz="0 1 0" />
         </joint>
@@ -158,6 +163,8 @@
             <child link="leg${leg_number}_link3" />
             <origin xyz="0 -${leg_link_y} 0" rpy="0 0 0" />
-            <limit lower="-${joint_limit}" upper="${joint_limit}"
-                effort="${joint_effort}" velocity="${joint_velocity}" />
+            <limit lower="${joint_lower_limit}"
+                   upper="${joint_upper_limit}"
+                   effort="${joint_effort_limit}"
+                   velocity="${joint_velocity_limit}" />
             <axis xyz="1 0 0" />
         </joint>

Commit message: Added comments to xacro property variables

File: robot/millihex.xacro (robot description, xacro)
@@ -2,21 +2,27 @@
 <robot xmlns:xacro="http://www.ros.org/wiki/xacro" name="millihex">
     <!-- Physical Properties -->
+    <!-- Torso mass and x,y dimensions -->
     <xacro:property name="torso_mass" value="0.01" />
     <xacro:property name="torso_x" value="0.14" />
     <xacro:property name="torso_y" value="0.04" />
+    <!-- Leg mass and x,y dimensions -->
     <xacro:property name="leg_link_mass" value="0.0008" />
     <xacro:property name="leg_link_x" value="0.02" />
     <xacro:property name="leg_link_y" value="0.03" />
+    <!-- Joint limits -->
     <xacro:property name="joint_upper_limit" value="1.5708" />
     <xacro:property name="joint_lower_limit" value="-1.5708" />
     <xacro:property name="joint_effort_limit" value="0.01" />
     <xacro:property name="joint_velocity_limit" value="0.01" />
+    <!-- Joint damping (b) and friction (k) -->
+    <xacro:property name="joint_damping" value="" />
+    <xacro:property name="joint_friction" value="" />
+    <!-- PCB thickness -->
     <xacro:property name="pcb_thickness_z" value="0.0005" />
+    <!-- Foot friction values -->
     <xacro:property name="foot_kp" value="1000.0" />
     <xacro:property name="foot_kd" value="1.0" />
     <xacro:property name="foot_mu1" value="0.5" />
     <xacro:property name="foot_mu2" value="0.5" />
-    <xacro:property name="joint_damping" value="" />
-    <xacro:property name="joint_friction" value="" />
     <!-- Color Definitions -->
     <material name="Black">

Commit message: Added dynamics elements to leg link joints in urdf

File: robot/millihex.xacro (robot description, xacro)
@@ -145,4 +145,5 @@
                    effort="${joint_effort_limit}"
                    velocity="${joint_velocity_limit}" />
+            <dynamics damping="${joint_damping}" friction="${joint_friction}" />
             <axis xyz="1 0 0" />
         </joint>
@@ -159,4 +160,5 @@
                    effort="${joint_effort_limit}"
                    velocity="${joint_velocity_limit}" />
+            <dynamics damping="${joint_damping}" friction="${joint_friction}" />
             <axis xyz="0 1 0" />
         </joint>
@@ -173,4 +175,5 @@
                    effort="${joint_effort_limit}"
                    velocity="${joint_velocity_limit}" />
+            <dynamics damping="${joint_damping}" friction="${joint_friction}" />
             <axis xyz="1 0 0" />
         </joint>
