Commit message: Dialing in Gazebo stiffness, damping, and friction coefficients

File: robot/millihex.xacro (robot description, xacro)
@@ -1,4 +1,4 @@
 <?xml version="1.0"?>
-<robot xmlns:xacro="http://www.ros.org/wiki/xacro" name="millihex">
+<robot name="millihex" xmlns:xacro="http://www.ros.org/wiki/xacro">
     <!-- Physical Properties -->
     <!-- Torso mass and x,y dimensions -->
@@ -16,13 +16,17 @@
     <xacro:property name="joint_velocity_limit" value="0.01" />
     <!-- Joint damping (b) and friction (k) -->
-    <xacro:property name="joint_damping" value="" />
-    <xacro:property name="joint_friction" value="" />
+    <xacro:property name="joint_damping" value="0.00003" />
+    <xacro:property name="joint_friction" value="0.001" />
     <!-- PCB thickness -->
     <xacro:property name="pcb_thickness_z" value="0.0005" />
-    <!-- Foot friction values -->
-    <xacro:property name="foot_kp" value="1000.0" />
-    <xacro:property name="foot_kd" value="1.0" />
-    <xacro:property name="foot_mu1" value="0.5" />
-    <xacro:property name="foot_mu2" value="0.5" />
+    <!-- Link Gazebo properties -->
+    <!-- Contact stiffness (kp) -->
+    <!-- Contact damping (kp) -->
+    <xacro:property name="link_kp" value="1000.0" />
+    <xacro:property name="link_kd" value="1000.0" />
+    <!-- Link coulomb friction coefficients in direction 1,2 -->
+    <!-- mu = [0, inf] where higher mu means less slip -->
+    <xacro:property name="link_mu1" value="5.0" />
+    <xacro:property name="link_mu2" value="5.0" />
     <!-- Color Definitions -->
     <material name="Black">
@@ -39,7 +43,6 @@
     <!-- Base and Torso Definition -->
     <xacro:macro name="millihex_torso" params="color">
-        <!-- Empty Base Link to attach robot to world -->
-        <link name="base_link">
-        </link>
+        <!-- Dummy link to support KDL -->
+        <link name="base_link" />
         <!-- Torso geometry without legs -->
         <link name="torso">
@@ -66,8 +69,8 @@
         <!-- Gazebo properties -->
         <gazebo reference="torso">
-            <kp>${foot_kp}</kp>
-            <kd>${foot_kd}</kd>
-            <mu1>${foot_mu1}</mu1>
-            <mu2>${foot_mu2}</mu2>
+            <kp>${link_kp}</kp>
+            <kd>${link_kd}</kd>
+            <mu1>${link_mu1}</mu1>
+            <mu2>${link_mu2}</mu2>
             <material>Gazebo/${color}</material>
         </gazebo>
@@ -105,8 +108,8 @@
         <!-- Gazebo properties -->
         <gazebo reference="leg${leg_number}_link${link_number}">
-            <kp>${foot_kp}</kp>
-            <kd>${foot_kd}</kd>
-            <mu1>${foot_mu1}</mu1>
-            <mu2>${foot_mu2}</mu2>
+            <kp>${link_kp}</kp>
+            <kd>${link_kd}</kd>
+            <mu1>${link_mu1}</mu1>
+            <mu2>${link_mu2}</mu2>
             <material>Gazebo/${color}</material>
         </gazebo>
@@ -141,9 +144,9 @@
             <child link="leg${leg_number}_link1" />
             <origin xyz="0 -${leg_link_y} 0" rpy="0 0 0" />
+            <dynamics damping="${joint_damping}" friction="${joint_friction}" />
             <limit lower="${joint_lower_limit}"
                    upper="${joint_upper_limit}"
                    effort="${joint_effort_limit}"
                    velocity="${joint_velocity_limit}" />
-            <dynamics damping="${joint_damping}" friction="${joint_friction}" />
             <axis xyz="1 0 0" />
         </joint>
@@ -156,9 +159,9 @@
             <child link="leg${leg_number}_link2" />
             <origin xyz="-${leg_link_y} 0 0" rpy="0 0 0" />
+            <dynamics damping="${joint_damping}" friction="${joint_friction}" />
             <limit lower="${joint_lower_limit}"
                    upper="${joint_upper_limit}"
                    effort="${joint_effort_limit}"
                    velocity="${joint_velocity_limit}" />
-            <dynamics damping="${joint_damping}" friction="${joint_friction}" />
             <axis xyz="0 1 0" />
         </joint>
@@ -171,9 +174,9 @@
             <child link="leg${leg_number}_link3" />
             <origin xyz="0 -${leg_link_y} 0" rpy="0 0 0" />
+            <dynamics damping="${joint_damping}" friction="${joint_friction}" />
             <limit lower="${joint_lower_limit}"
                    upper="${joint_upper_limit}"
                    effort="${joint_effort_limit}"
                    velocity="${joint_velocity_limit}" />
-            <dynamics damping="${joint_damping}" friction="${joint_friction}" />
             <axis xyz="1 0 0" />
         </joint>

Commit message: Added robot_stance method in Robot class to make millihex stand up. Also reversed direction of leg joint 2 axis to make control angle direction the same as leg joints 1 and 3

File: robot/millihex.xacro (robot description, xacro)
@@ -164,5 +164,5 @@
                    effort="${joint_effort_limit}"
                    velocity="${joint_velocity_limit}" />
-            <axis xyz="0 1 0" />
+            <axis xyz="0 -1 0" />
         </joint>
         <xacro:leg_transmission leg_number="${leg_number}" joint_number="2" />

Commit message: Doubled coulomb friction for robot so that it does not go through the floor

File: robot/millihex.xacro (robot description, xacro)
@@ -27,6 +27,6 @@
     <!-- Link coulomb friction coefficients in direction 1,2 -->
     <!-- mu = [0, inf] where higher mu means less slip -->
-    <xacro:property name="link_mu1" value="5.0" />
-    <xacro:property name="link_mu2" value="5.0" />
+    <xacro:property name="link_mu1" value="10.0" />
+    <xacro:property name="link_mu2" value="10.0" />
     <!-- Color Definitions -->
     <material name="Black">
